File: hardware/BlackBodyBoard.kicad_sch (KiCad schematic)
At the start: 19 parts, among them J10 CAN_OUT, J4 CAN_DEBUG, J5 CAN_IN

Commit message: irradescence stuff
Parts:
- removed F1: Fuse, symbol Device:Fuse
- removed J10: CAN_OUT, LHRS_Connectors:Molex_Nano-Fit_105309-xx05_1x05_P2.50mm_Vertical, symbol lhrs_connectors:CAN_NANO_01x05
- removed J4: CAN_DEBUG, Connector_Molex:Molex_Nano-Fit_105309-xx04_1x04_P2.50mm_Vertical, symbol lhrs_connectors:CAN_DEBUG_NANO_01x04
- removed J5: CAN_IN, LHRS_Connectors:Molex_Nano-Fit_105309-xx05_1x05_P2.50mm_Vertical, symbol lhrs_connectors:CAN_NANO_01x05
- removed JP2: SolderJumper_2_Open, symbol Jumper:SolderJumper_2_Open
- removed R59: 0, symbol Device:R
- removed R64: 16kR, symbol Device:R
- removed R65: 4.7kR, symbol Device:R
- removed TP17: Power TestPoint, symbol Connector:TestPoint
- removed TP18: MCU TestPoint, symbol Connector:TestPoint
- removed TP19: CAN TestPoint, symbol Connector:TestPoint
- removed TP20, TP21, TP22, TP23, TP24: TestPoint, symbol Connector:TestPoint
- removed TP25: LDO_OUT_TestPoint, symbol Connector:TestPoint
- added D14, D15: LED, LED_SMD:LED_0603_1608Metric, symbol lhrs_misc:Blue_LED
- added F2: Fuse, symbol Device:Fuse
- added J11: CAN_OUT, LHRS_Connectors:Molex_Nano-Fit_105309-xx05_1x05_P2.50mm_Vertical, symbol lhrs_connectors:CAN_NANO_01x05
- added J6: CAN_DEBUG, Connector_Molex:Molex_Nano-Fit_105309-xx04_1x04_P2.50mm_Vertical, symbol lhrs_connectors:CAN_DEBUG_NANO_01x04
- added J7: CAN_IN, LHRS_Connectors:Molex_Nano-Fit_105309-xx05_1x05_P2.50mm_Vertical, symbol lhrs_connectors:CAN_NANO_01x05
- added JP3: SolderJumper_2_Open, symbol Jumper:SolderJumper_2_Open
- added R30, R31: 1k, symbol Device:R
- added R41, R42, R48: 22, symbol Device:R
- added R60, R61: 0, symbol Device:R
- added R66: 16k, symbol Device:R
- added R67: 4.7k, symbol Device:R
- added TP38: +12V, symbol Connector:TestPoint
- added TP39: +12V_PP, symbol Connector:TestPoint
- added TP40: +5V_BUCK, symbol Connector:TestPoint
- added TP41: +USBC_5V, symbol Connector:TestPoint
- added TP42: MUX_OUT, symbol Connector:TestPoint
- added TP43: LDO_OUT_TestPoint, symbol Connector:TestPoint
- added TP44: Power TestPoint, symbol Connector:TestPoint
- added TP45: MCU TestPoint, symbol Connector:TestPoint
- added TP46: CAN TestPoint, symbol Connector:TestPoint
- added TP47: SPI_MISO, symbol Connector:TestPoint
- added TP48: SPI_MOSI, symbol Connector:TestPoint
- added TP49: SPI_SCK, symbol Connector:TestPoint
Connections:
- net +12V: now also F2.1, J11.1 (12V), J6.1 (12V), J7.1 (12V), TP38.1
- net +12V_PP: now also JP3.2 (B), TP39.1
- net +3.3V: now also TP43.1
- net +5V_BUCK: now also R66.1, TP40.1
- net +USBC_5V: now also TP41.1
- net 48PinMCU/PB6: now also R31.1
- net 48PinMCU/PB7: now also R30.1
- net CAN_H: now also J6.2 (CAN_H), J7.2 (CAN_H)
- net CAN_L: now also J6.3 (CAN_L), J7.3 (CAN_L)
- net GND: now also D14.1 (K), D15.1 (K), J11.4 (GND), J6.4 (GND), J7.4 (GND), R60.2, R61.2, R67.2, TP44.1, TP45.1, TP46.1
- net SPI_MISO: now also R42.2, TP47.1
- net SPI_MOSI: now also R41.2, TP48.1
- net SPI_SCK: now also R48.2, TP49.1
- new net: J7.5 (SHIELD), R60.1
- new net: J11.5 (SHIELD), R61.1
- new net: D15.2 (A), R31.2
- new net: D14.2 (A), R30.2
- new net +5V: TP42.1
- new net 48PinMCU/PA5: R48.1
- new net 48PinMCU/PA6: R42.1
- new net 48PinMCU/PA7: R41.1
- new net PowerProtection1/Vin: F2.2, JP3.1 (A)
- new net Power_Mux1/PR1: R66.2, R67.1
- no-connect marks 21 -> 19
Other:
- removed sheet 12VBuck
- removed sheet LDO 3.3V
- removed sheet PowerProtection
- removed sheet Power_Mux
- added sheet 12VBuck1 (12VBuck.kicad_sch)
- added sheet LDO 3.3V1 (LDO.kicad_sch)
- added sheet PowerProtection1 (PowerProtection.kicad_sch)
- added sheet Power_Mux1 (Power_Mux.kicad_sch)
- company: Longhorn Racing Solar - VCAT Telemetry -> (none)
- title: Blackbody Board -> (none)
