File: hardware/BlackBodyBoard.kicad_sch (KiCad schematic)
At the start: 30 parts, among them J11 CAN_OUT, J6 CAN_DEBUG, J7 CAN_IN

Commit message: check breakout board layout
Connections:
- net CAN_H: now also J11.2 (CAN_H)
- net CAN_L: now also J11.3 (CAN_L)
- net +5V renamed MUX_OUT
Other:
- sheet 48PinMCU ports: added none; removed VDDA
- sheet Irradiance ports: added I2C_SCL, I2C_SDA, IRRAD_INT; removed GNDA, IRRAD_ADC, IRRAD_DET, IRRAD_TEST, VDDA
