File: hardware/BlackBodyBoard.kicad_sch (KiCad schematic)
At the start: 30 parts, among them J11 CAN_OUT, J6 CAN_DEBUG, J7 CAN_IN

Commit message: Main board placement + silkscreen, breakout ground plane, DRC rule updates
- Grouped placement and condensed outline (2 mm rounded corners)
- Silkscreen refs moved next to their parts, pin labels added
- Interrupt removed from main board and breakout (test point instead)
- Breakout: B.Cu ground plane + stitching vias
- Default clearance / hole clearance lowered to 0.15 mm
Parts:
- F2: footprint (none) -> LHRS_Power:Fuse-3557-2; LCSC P/N (none) -> C352820; P/N (none) -> 3557-2
- JP3: footprint (none) -> Jumper:SolderJumper-2_P1.3mm_Open_RoundedPad1.0x1.5mm
- R29, R30, R31: footprint (none) -> Resistor_SMD:R_0603_1608Metric_Pad0.98x0.95mm_HandSolder; LCSC P/N (none) -> C21190; P/N (none) -> 0603WAF1001T5E
- R41, R42, R48: footprint (none) -> Resistor_SMD:R_0603_1608Metric_Pad0.98x0.95mm_HandSolder; LCSC P/N (none) -> C2930077; P/N (none) -> FRC0603F22R0TS
- R60, R61: footprint (none) -> Resistor_SMD:R_0603_1608Metric_Pad0.98x0.95mm_HandSolder; LCSC P/N (none) -> C21189; P/N (none) -> CRCW06030000Z0EE
- R66: footprint (none) -> Resistor_SMD:R_0603_1608Metric_Pad0.98x0.95mm_HandSolder; LCSC P/N (none) -> C22818; P/N (none) -> 0603WAF1602T5E
- R67: footprint (none) -> Resistor_SMD:R_0603_1608Metric_Pad0.98x0.95mm_HandSolder; LCSC P/N (none) -> C23162; P/N (none) -> 0603WAF4701T5E
- TP38, TP39, TP40, TP41, TP42, TP43, TP44, TP45, TP46, TP47, TP48, TP49: footprint (none) -> TestPoint:TestPoint_Pad_D1.5mm
Connections:
- no-connect marks 19 -> 20
Other:
- sheet Irradiance ports: added none; removed IRRAD_INT
