File: hardware/LDO.kicad_sch (KiCad schematic)
At the start: 5 parts, among them U2 MCP1826S

Commit message: irradescence stuff
Parts:
- renumbered C20 to C46, C21 to C47, D5 to D10, TP_3.3V1 to TP_3.3V2, U2 to U6
Changed lines of the file:
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@@
 		(dnp no)
 		(fields_autoplaced yes)
-		(property "Reference" "C21"
+		(property "Reference" "C47"
 			(at 168.275 68.5735 0)
 			(show_name no)
@@
 		)
 		(instances
+			(project "BlackBodyBoard"
+				(path "/48096f47-ddef-4ea4-8e15-14613f1872f0/8469fd14-d805-40d8-82a1-d1c2e1c25361"
+					(reference "C47")
+					(unit 1)
+				)
+			)
 			(project "LDO"
 				(path "/8ff43370-8d10-4d2c-b1a3-81d1c2934a98"
@@
 				(path "/e5b32072-3e3d-42a6-9d41-1a76d538e329/f3053c74-1ac6-4a33-80f3-565e8c4c2c7d"
 					(reference "C?")
-					(unit 1)
-				)
-			)
-			(project "BlackBodyBoard"
-				(path "/48096f47-ddef-4ea4-8e15-14613f1872f0/742608da-0aa6-442d-97ae-43bdb3ce7e6a"
-					(reference "C21")
 					(unit 1)
 				)
@@
 		(in_pos_files yes)
 		(dnp no)
-		(property "Reference" "TP_3.3V1"
+		(property "Reference" "TP_3.3V2"
 			(at 166.624 54.356 90)
 			(show_name no)
@@
 		)
 		(instances
+			(project "BlackBodyBoard"
+				(path "/48096f47-ddef-4ea4-8e15-14613f1872f0/8469fd14-d805-40d8-82a1-d1c2e1c25361"
+					(reference "TP_3.3V2")
+					(unit 1)
+				)
+			)
 			(project "LDO"
 				(path "/8ff43370-8d10-4d2c-b1a3-81d1c2934a98"
-					(reference "TP_3.3V1")
-					(unit 1)
-				)
-			)
-			(project "BlackBodyBoard"
-				(path "/48096f47-ddef-4ea4-8e15-14613f1872f0/742608da-0aa6-442d-97ae-43bdb3ce7e6a"
 					(reference "TP_3.3V1")
 					(unit 1)
@@
 		(dnp no)
 		(fields_autoplaced yes)
-		(property "Reference" "U2"
+		(property "Reference" "U6"
 			(at 152.4 56.515 0)
 			(show_name no)
@@
 		)
 		(instances
+			(project "BlackBodyBoard"
+				(path "/48096f47-ddef-4ea4-8e15-14613f1872f0/8469fd14-d805-40d8-82a1-d1c2e1c25361"
+					(reference "U6")
+					(unit 1)
+				)
+			)
 			(project ""
 				(path "/8ff43370-8d10-4d2c-b1a3-81d1c2934a98"
 					(reference "U1")
-					(unit 1)
-				)
-			)
-			(project "BlackBodyBoard"
-				(path "/48096f47-ddef-4ea4-8e15-14613f1872f0/742608da-0aa6-442d-97ae-43bdb3ce7e6a"
-					(reference "U2")
 					(unit 1)
 				)
@@
 		(dnp no)
 		(fields_autoplaced yes)
-		(property "Reference" "#FLG09"
+		(property "Reference" "#FLG016"
 			(at 142.24 65.405 0)
 			(hide yes)
@@
 		(instances
 			(project "BlackBodyBoard"
-				(path "/48096f47-ddef-4ea4-8e15-14613f1872f0/742608da-0aa6-442d-97ae-43bdb3ce7e6a"
-					(reference "#FLG09")
+				(path "/48096f47-ddef-4ea4-8e15-14613f1872f0/8469fd14-d805-40d8-82a1-d1c2e1c25361"
+					(reference "#FLG016")
 					(unit 1)
 				)
@@
 		(dnp no)
 		(fields_autoplaced yes)
-		(property "Reference" "D5"
+		(property "Reference" "D10"
 			(at 133.604 57.15 0)
 			(show_name no)
@@
 		)
 		(instances
+			(project "BlackBodyBoard"
+				(path "/48096f47-ddef-4ea4-8e15-14613f1872f0/8469fd14-d805-40d8-82a1-d1c2e1c25361"
+					(reference "D10")
+					(unit 1)
+				)
+			)
 			(project ""
 				(path "/8ff43370-8d10-4d2c-b1a3-81d1c2934a98"
 					(reference "D1")
-					(unit 1)
-				)
-			)
-			(project "BlackBodyBoard"
-				(path "/48096f47-ddef-4ea4-8e15-14613f1872f0/742608da-0aa6-442d-97ae-43bdb3ce7e6a"
-					(reference "D5")
 					(unit 1)
 				)
@@
 		(dnp no)
 		(fields_autoplaced yes)
-		(property "Reference" "C20"
+		(property "Reference" "C46"
 			(at 142.875 68.5735 0)
 			(show_name no)
@@
 		)
 		(instances
+			(project "BlackBodyBoard"
+				(path "/48096f47-ddef-4ea4-8e15-14613f1872f0/8469fd14-d805-40d8-82a1-d1c2e1c25361"
+					(reference "C46")
+					(unit 1)
+				)
+			)
 			(project "LDO"
 				(path "/8ff43370-8d10-4d2c-b1a3-81d1c2934a98"
@@
 					(unit 1)
 				)
-			)
-			(project "BlackBodyBoard"
-				(path "/48096f47-ddef-4ea4-8e15-14613f1872f0/742608da-0aa6-442d-97ae-43bdb3ce7e6a"
-					(reference "C20")
-					(unit 1)
-				)
