File: hardware/12VBuck.kicad_sch (KiCad schematic)
At the start: 14 parts, among them U3 LMR51635XDDCR

Commit message: irradescence stuff
Parts:
- removed TP2: CB, TestPoint:TestPoint_THTPad_D3.0mm_Drill1.5mm, symbol Connector:TestPoint
- removed TP3: FB, TestPoint:TestPoint_THTPad_D3.0mm_Drill1.5mm, symbol Connector:TestPoint
- removed TP4: SW, TestPoint:TestPoint_THTPad_D3.0mm_Drill1.5mm, symbol Connector:TestPoint
- TP5: renamed from TP1; footprint TestPoint:TestPoint_THTPad_D3.0mm_Drill1.5mm -> Connector_PinHeader_2.54mm:PinHeader_1x01_P2.54mm_Vertical
- renumbered C34 to C40, C35 to C41, C36 to C42, C37 to C43, C38 to C44, C39 to C45, L1 to L2, R20 to R22, R21 to R23, U3 to U5

Commit message: check breakout board layout
Parts:
- U5: footprint (none) -> LHRS_ICs:DDC0006A-MFG
Changed lines of the file:
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@@
 			)
 		)
-		(property "Footprint" ""
+		(property "Footprint" "LHRS_ICs:DDC0006A-MFG"
 			(at 114.3 81.28 0)
 			(hide yes)
