File: hardware/48PinMCU.kicad_sch (KiCad schematic)
At the start: 34 parts, among them J1 SWD_Header, J2 SWD, SW1 Reset, SW2 SW_SPDT, U1 STM32G473CETx, Y1 Crystal

Commit message: irradescence stuff
Parts:
- added C?: 10u, Capacitor_SMD:C_0603_1608Metric_Pad1.08x0.95mm_HandSolder, symbol Device:C
- C10, C12, C13, C14, C3, C5, C6, C7, C8: value 0.1uF -> 0.1u
- C11, C9: value 1uF -> 1u
- C15: value 100nF -> 100n
- C4: value 10uF -> 10u
Connections:
- net GNDA: now also C?.2
- net VDDA: now also C?.1
Other:
- note added: "What do I do now thatr i have 4 channels thins kinda means 40mA all flow thorugh the ferrite bead can you explain what to do?"

Commit message: check breakout board layout
Parts:
- J1: symbol 100PinMCU:SWD_Header_02x02 -> lhrs_connectors:SWD_Header_02x02
- gave numbers to parts that had none: 1
Changed lines of the file:
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@@
+		)
+	)
+	(label "VDDA"
+		(at 80.01 17.78 180)
+		(effects
+			(font
+				(size 1.27 1.27)
+			)
+			(justify right bottom)
 		)
 	)
@@
 		)
 	)
+	(label "VDDA"
+		(at 259.08 54.61 0)
+		(effects
+			(font
+				(size 1.27 1.27)
+			)
+			(justify left bottom)
+		)
+	)
 	(label "PA2"
 		(at 132.08 41.91 0)
+		(effects
+			(font
+				(size 1.27 1.27)
+			)
+			(justify left bottom)
+		)
+	)
+	(label "VDDA"
+		(at 196.85 48.26 0)
 		(effects
 			(font
@@
 		)
 	)
-	(hierarchical_label "VDDA"
-		(shape input)
-		(at 80.01 17.78 180)
-		(effects
-			(font
-				(size 1.27 1.27)
-			)
-			(justify right)
-		)
-	)
 	(hierarchical_label "NRST"
 		(shape input)
@@
 		)
 	)
-	(hierarchical_label "VDDA"
-		(shape input)
-		(at 259.08 54.61 0)
-		(effects
-			(font
-				(size 1.27 1.27)
-			)
-			(justify left)
-		)
-	)
 	(hierarchical_label "+3V3"
 		(shape input)
@@
 		(shape bidirectional)
 		(at 121.92 49.53 0)
-		(effects
-			(font
-				(size 1.27 1.27)
-			)
-			(justify left)
-		)
-	)
-	(hierarchical_label "VDDA"
-		(shape input)
-		(at 196.85 48.26 0)
 		(effects
 			(font
@@
 	)
 	(symbol
-		(lib_id "100PinMCU:SWD_Header_02x02")
+		(lib_id "lhrs_connectors:SWD_Header_02x02")
 		(at 247.65 133.35 0)
 		(unit 1)
@@
 		(in_pos_files yes)
 		(dnp no)
-		(property "Reference" "C?"
+		(property "Reference" "C59"
 			(at 226.568 56.388 0)
 			(show_name no)
@@
 			(project "BlackBodyBoard"
 				(path "/48096f47-ddef-4ea4-8e15-14613f1872f0/cc54fbd4-47b5-4c2e-a438-64ef2059228d"
-					(reference "C?")
+					(reference "C59")
 					(unit 1)
 				)
