File: hardware/CAN_Transceiver.kicad_sch (KiCad schematic)
At the start: 9 parts, among them IC1 TCAN3413DR

Commit message: check breakout board layout
Parts:
- C19: symbol ECE319K:C -> Device:C
- D4: symbol CDSOT23-T24CAN:CDSOT23-T24CAN -> lhrs_misc:CDSOT23-T24CAN
- IC1: symbol TCAN3413DR:TCAN3413DR -> lhrs_ics:TCAN3413DR
Changed lines of the file:
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@@
 	)
 	(symbol
-		(lib_id "ECE319K:C")
+		(lib_id "Device:C")
 		(at 189.23 88.9 180)
 		(unit 1)
@@
 	)
 	(symbol
-		(lib_id "CDSOT23-T24CAN:CDSOT23-T24CAN")
+		(lib_id "lhrs_misc:CDSOT23-T24CAN")
 		(at 185.42 54.61 0)
 		(unit 1)
@@
 	)
 	(symbol
-		(lib_id "TCAN3413DR:TCAN3413DR")
+		(lib_id "lhrs_ics:TCAN3413DR")
 		(at 111.76 71.12 0)
 		(unit 1)
