File: hardware/PowerProtection.kicad_sch (KiCad schematic)
At the start: 18 parts, among them IC2 LM74502DDFR, Q1 PSMN012-100YS, Q2 PSMN012-100YS

Commit message: irradescence stuff
Parts:
- renumbered C22 to C48, C23 to C49, C29 to C50, C30 to C51, C31 to C52, C32 to C53, C33 to C54, D6 to D11, D9 to D12, IC2 to IC3, Q1 to Q3, Q2 to Q4, R14 to R24, R15 to R25, R16 to R26, R17 to R27, R18 to R28, R19 to R32

Commit message: check breakout board layout
Parts:
- C51: symbol ECE319H:C -> Device:C
Changed lines of the file:
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@@
 	)
 	(symbol
-		(lib_id "ECE319H:C")
+		(lib_id "Device:C")
 		(at 60.96 63.5 0)
 		(unit 1)
