File: hardware/Power_Mux.kicad_sch (KiCad schematic)
At the start: 6 parts, among them U4 TPS2117DRLR

Commit message: irradescence stuff
Parts:
- C55: renamed from C25; value 0.1uF -> 0.1u
- C56: renamed from C26; value 0.1uF -> 0.1u
- C57: renamed from C27; value 0.1uF -> 0.1u
- C58: renamed from C28; value 0.1uF -> 0.1u
- renumbered R13 to R33, U4 to U7
Changed lines of the file:
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@@
 		(in_pos_files yes)
 		(dnp no)
-		(property "Reference" "C28"
+		(property "Reference" "C58"
 			(at 91.8972 57.2516 0)
 			(show_name no)
@@
 			)
 		)
-		(property "Value" "0.1uF"
+		(property "Value" "0.1u"
 			(at 91.8972 59.563 0)
 			(show_name no)
@@
 		)
 		(instances
+			(project "BlackBodyBoard"
+				(path "/48096f47-ddef-4ea4-8e15-14613f1872f0/6222ccd3-d1ee-4d0b-8dcb-c263153f217a"
+					(reference "C58")
+					(unit 1)
+				)
+			)
 			(project "power-mux-block"
 				(path "/c8207045-8aef-4538-bcc4-1e380c549c2c"
 					(reference "C4")
-					(unit 1)
-				)
-			)
-			(project "BlackBodyBoard"
-				(path "/48096f47-ddef-4ea4-8e15-14613f1872f0/ad2265c7-0a96-4914-a6f0-818e23817a72"
-					(reference "C28")
 					(unit 1)
 				)
@@
 		(in_pos_files yes)
 		(dnp no)
-		(property "Reference" "R13"
+		(property "Reference" "R33"
 			(at 78.994 67.564 0)
 			(show_name no)
@@
 		)
 		(instances
+			(project "BlackBodyBoard"
+				(path "/48096f47-ddef-4ea4-8e15-14613f1872f0/6222ccd3-d1ee-4d0b-8dcb-c263153f217a"
+					(reference "R33")
+					(unit 1)
+				)
+			)
 			(project "power-mux-block"
 				(path "/c8207045-8aef-4538-bcc4-1e380c549c2c"
 					(reference "R1")
-					(unit 1)
-				)
-			)
-			(project "BlackBodyBoard"
-				(path "/48096f47-ddef-4ea4-8e15-14613f1872f0/ad2265c7-0a96-4914-a6f0-818e23817a72"
-					(reference "R13")
 					(unit 1)
 				)
@@
 		(in_pos_files yes)
 		(dnp no)
-		(property "Reference" "C25"
+		(property "Reference" "C55"
 			(at 24.5872 44.5516 0)
 			(show_name no)
@@
 			)
 		)
-		(property "Value" "0.1uF"
+		(property "Value" "0.1u"
 			(at 24.5872 46.863 0)
 			(show_name no)
@@
 		)
 		(instances
+			(project "BlackBodyBoard"
+				(path "/48096f47-ddef-4ea4-8e15-14613f1872f0/6222ccd3-d1ee-4d0b-8dcb-c263153f217a"
+					(reference "C55")
+					(unit 1)
+				)
+			)
 			(project "power-mux-block"
 				(path "/c8207045-8aef-4538-bcc4-1e380c549c2c"
 					(reference "C1")
-					(unit 1)
-				)
-			)
-			(project "BlackBodyBoard"
-				(path "/48096f47-ddef-4ea4-8e15-14613f1872f0/ad2265c7-0a96-4914-a6f0-818e23817a72"
-					(reference "C25")
 					(unit 1)
 				)
@@
 		(dnp no)
 		(fields_autoplaced yes)
-		(property "Reference" "U4"
+		(property "Reference" "U7"
 			(at 60.96 44.45 0)
 			(show_name no)
@@
 		)
 		(instances
+			(project "BlackBodyBoard"
+				(path "/48096f47-ddef-4ea4-8e15-14613f1872f0/6222ccd3-d1ee-4d0b-8dcb-c263153f217a"
+					(reference "U7")
+					(unit 1)
+				)
+			)
 			(project ""
 				(path "/c8207045-8aef-4538-bcc4-1e380c549c2c"
 					(reference "U1")
-					(unit 1)
-				)
-			)
-			(project "BlackBodyBoard"
-				(path "/48096f47-ddef-4ea4-8e15-14613f1872f0/ad2265c7-0a96-4914-a6f0-818e23817a72"
-					(reference "U4")
 					(unit 1)
 				)
@@
 		(in_pos_files yes)
 		(dnp no)
-		(property "Reference" "C27"
+		(property "Reference" "C57"
 			(at 42.3672 67.4116 0)
 			(show_name no)
@@
 			)
 		)
-		(property "Value" "0.1uF"
+		(property "Value" "0.1u"
 			(at 42.3672 69.723 0)
 			(show_name no)
@@
 		)
 		(instances
+			(project "BlackBodyBoard"
+				(path "/48096f47-ddef-4ea4-8e15-14613f1872f0/6222ccd3-d1ee-4d0b-8dcb-c263153f217a"
+					(reference "C57")
+					(unit 1)
+				)
+			)
 			(project "power-mux-block"
 				(path "/c8207045-8aef-4538-bcc4-1e380c549c2c"
 					(reference "C3")
-					(unit 1)
-				)
-			)
-			(project "BlackBodyBoard"
-				(path "/48096f47-ddef-4ea4-8e15-14613f1872f0/ad2265c7-0a96-4914-a6f0-818e23817a72"
-					(reference "C27")
 					(unit 1)
 				)
@@
 		(in_pos_files yes)
 		(dnp no)
-		(property "Reference" "C26"
+		(property "Reference" "C56"
 			(at 38.5572 44.5516 0)
 			(show_name no)
@@
 			)
 		)
-		(property "Value" "0.1uF"
+		(property "Value" "0.1u"
 			(at 38.5572 46.863 0)
 			(show_name no)
@@
 		)
 		(instances
+			(project "BlackBodyBoard"
+				(path "/48096f47-ddef-4ea4-8e15-14613f1872f0/6222ccd3-d1ee-4d0b-8dcb-c263153f217a"
+					(reference "C56")
+					(unit 1)
+				)
+			)
 			(project "power-mux-block"
 				(path "/c8207045-8aef-4538-bcc4-1e380c549c2c"
@@
 					(unit 1)
 				)
-			)
-			(project "BlackBodyBoard"
-				(path "/48096f47-ddef-4ea4-8e15-14613f1872f0/ad2265c7-0a96-4914-a6f0-818e23817a72"
-					(reference "C26")
-					(unit 1)
-				)

Commit message: check breakout board layout
Parts:
- U7: symbol mux:TPS2117DRLR -> lhrs_ics:TPS2117DRLR
Changed lines of the file:
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@@
 	)
 	(symbol
-		(lib_id "mux:TPS2117DRLR")
+		(lib_id "lhrs_ics:TPS2117DRLR")
 		(at 60.96 62.23 0)
 		(unit 1)
