File: hardware/USB-C_Connector.kicad_sch (KiCad schematic)
At the start: 6 parts, among them J3 USB_C_Receptacle_USB2.0_16P

Commit message: irradescence stuff
Parts:
- C24: value 10uF -> 10u
Changed lines of the file:
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@@
 		)
 		(instances
+			(project "BlackBodyBoard"
+				(path "/48096f47-ddef-4ea4-8e15-14613f1872f0/3e1f507b-ac4b-41d9-a5aa-5ad5a924ba8f"
+					(reference "R11")
+					(unit 1)
+				)
+			)
 			(project "usb_conn"
 				(path "/64d5c21e-b85c-41ec-b08c-3556f1a0ecf2"
 					(reference "R1")
-					(unit 1)
-				)
-			)
-			(project "BlackBodyBoard"
-				(path "/48096f47-ddef-4ea4-8e15-14613f1872f0/3e1f507b-ac4b-41d9-a5aa-5ad5a924ba8f"
-					(reference "R11")
 					(unit 1)
 				)
@@
 		)
 		(instances
+			(project "BlackBodyBoard"
+				(path "/48096f47-ddef-4ea4-8e15-14613f1872f0/3e1f507b-ac4b-41d9-a5aa-5ad5a924ba8f"
+					(reference "R12")
+					(unit 1)
+				)
+			)
 			(project "usb_conn"
 				(path "/64d5c21e-b85c-41ec-b08c-3556f1a0ecf2"
 					(reference "R2")
-					(unit 1)
-				)
-			)
-			(project "BlackBodyBoard"
-				(path "/48096f47-ddef-4ea4-8e15-14613f1872f0/3e1f507b-ac4b-41d9-a5aa-5ad5a924ba8f"
-					(reference "R12")
 					(unit 1)
 				)
@@
 		)
 		(instances
+			(project "BlackBodyBoard"
+				(path "/48096f47-ddef-4ea4-8e15-14613f1872f0/3e1f507b-ac4b-41d9-a5aa-5ad5a924ba8f"
+					(reference "J3")
+					(unit 1)
+				)
+			)
 			(project "usb_conn"
 				(path "/64d5c21e-b85c-41ec-b08c-3556f1a0ecf2"
 					(reference "J1")
-					(unit 1)
-				)
-			)
-			(project "BlackBodyBoard"
-				(path "/48096f47-ddef-4ea4-8e15-14613f1872f0/3e1f507b-ac4b-41d9-a5aa-5ad5a924ba8f"
-					(reference "J3")
 					(unit 1)
 				)
@@
 		)
 		(instances
+			(project "BlackBodyBoard"
+				(path "/48096f47-ddef-4ea4-8e15-14613f1872f0/3e1f507b-ac4b-41d9-a5aa-5ad5a924ba8f"
+					(reference "#FLG01")
+					(unit 1)
+				)
+			)
 			(project "usb_conn"
 				(path "/64d5c21e-b85c-41ec-b08c-3556f1a0ecf2"
-					(reference "#FLG01")
-					(unit 1)
-				)
-			)
-			(project "BlackBodyBoard"
-				(path "/48096f47-ddef-4ea4-8e15-14613f1872f0/3e1f507b-ac4b-41d9-a5aa-5ad5a924ba8f"
 					(reference "#FLG01")
 					(unit 1)
@@
 		)
 		(instances
+			(project "BlackBodyBoard"
+				(path "/48096f47-ddef-4ea4-8e15-14613f1872f0/3e1f507b-ac4b-41d9-a5aa-5ad5a924ba8f"
+					(reference "D7")
+					(unit 1)
+				)
+			)
 			(project "usb_conn"
 				(path "/64d5c21e-b85c-41ec-b08c-3556f1a0ecf2"
 					(reference "D1")
-					(unit 1)
-				)
-			)
-			(project "BlackBodyBoard"
-				(path "/48096f47-ddef-4ea4-8e15-14613f1872f0/3e1f507b-ac4b-41d9-a5aa-5ad5a924ba8f"
-					(reference "D7")
 					(unit 1)
 				)
@@
 			)
 		)
-		(property "Value" "10uF"
+		(property "Value" "10u"
 			(at 64.3128 35.687 0)
 			(show_name no)
@@
 		)
 		(instances
+			(project "BlackBodyBoard"
+				(path "/48096f47-ddef-4ea4-8e15-14613f1872f0/3e1f507b-ac4b-41d9-a5aa-5ad5a924ba8f"
+					(reference "C24")
+					(unit 1)
+				)
+			)
 			(project "usb_conn"
 				(path "/64d5c21e-b85c-41ec-b08c-3556f1a0ecf2"
 					(reference "C1")
-					(unit 1)
-				)
-			)
-			(project "BlackBodyBoard"
-				(path "/48096f47-ddef-4ea4-8e15-14613f1872f0/3e1f507b-ac4b-41d9-a5aa-5ad5a924ba8f"
-					(reference "C24")
 					(unit 1)
 				)
@@
 		)
 		(instances
+			(project "BlackBodyBoard"
+				(path "/48096f47-ddef-4ea4-8e15-14613f1872f0/3e1f507b-ac4b-41d9-a5aa-5ad5a924ba8f"
+					(reference "D8")
+					(unit 1)
+				)
+			)
 			(project "usb_conn"
 				(path "/64d5c21e-b85c-41ec-b08c-3556f1a0ecf2"
@@
 					(unit 1)
 				)
-			)
-			(project "BlackBodyBoard"
-				(path "/48096f47-ddef-4ea4-8e15-14613f1872f0/3e1f507b-ac4b-41d9-a5aa-5ad5a924ba8f"
-					(reference "D8")
-					(unit 1)
-				)

Commit message: check breakout board layout
Parts:
- J3: footprint LHRS_ICs:USB_C_Receptacle_GCT_USB4105-xx-A_16P_TopMnt_Horizontal -> LHRS_Connectors:USB_C_Receptacle_GCT_USB4105-xx-A_16P_TopMnt_Horizontal
Changed lines of the file:
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@@
 			)
 		)
-		(property "Footprint" "LHRS_ICs:USB_C_Receptacle_GCT_USB4105-xx-A_16P_TopMnt_Horizontal"
+		(property "Footprint" "LHRS_Connectors:USB_C_Receptacle_GCT_USB4105-xx-A_16P_TopMnt_Horizontal"
 			(at 39.37 45.72 0)
 			(hide yes)
