File: hardware/BlackBodyBoard.kicad_pcb (KiCad board)
At the start: 0 parts

Commit message: Main board placement + silkscreen, breakout ground plane, DRC rule updates
- Grouped placement and condensed outline (2 mm rounded corners)
- Silkscreen refs moved next to their parts, pin labels added
- Interrupt removed from main board and breakout (test point instead)
- Breakout: B.Cu ground plane + stitching vias
- Default clearance / hole clearance lowered to 0.15 mm
Parts:
- added C1: 26p, Capacitor_SMD:C_0603_1608Metric_Pad1.08x0.95mm_HandSolder, F.Cu at (155.7, 77.1)
- added C10: 0.1u, Capacitor_SMD:C_0603_1608Metric_Pad1.08x0.95mm_HandSolder, F.Cu at (161.4, 72.7)
- added C11: 1u, Capacitor_SMD:C_0603_1608Metric_Pad1.08x0.95mm_HandSolder, F.Cu at (172.4, 90.6)
- added C12: 0.1u, Capacitor_SMD:C_0603_1608Metric_Pad1.08x0.95mm_HandSolder, F.Cu at (159.8, 74.5)
- added C13: 0.1u, Capacitor_SMD:C_0603_1608Metric_Pad1.08x0.95mm_HandSolder, F.Cu at (174.1, 74.9)
- added C14: 0.1u, Capacitor_SMD:C_0603_1608Metric_Pad1.08x0.95mm_HandSolder, F.Cu at (163.9, 71.9)
- added C15: 100n, Capacitor_SMD:C_0603_1608Metric_Pad1.08x0.95mm_HandSolder, F.Cu at (170.2, 94.3)
- added C16: 10u, Capacitor_SMD:C_0805_2012Metric_Pad1.18x1.45mm_HandSolder, F.Cu at (171.3, 99.5)
- added C17: 0.1u, Capacitor_SMD:C_0603_1608Metric_Pad1.08x0.95mm_HandSolder, F.Cu at (174.9, 88.6)
- added C18: 0.1u, Capacitor_SMD:C_0603_1608Metric_Pad1.08x0.95mm_HandSolder, F.Cu at (170.6, 91.7)
- added C19: 0.1u, Capacitor_SMD:C_0603_1608Metric_Pad1.08x0.95mm_HandSolder, F.Cu at (172.8, 94.6)
- added C2: 26p, Capacitor_SMD:C_0603_1608Metric_Pad1.08x0.95mm_HandSolder, F.Cu at (155.7, 80.6)
- added C23: 100n, Capacitor_SMD:C_0603_1608Metric_Pad1.08x0.95mm_HandSolder, F.Cu at (164.3, 94.6)
- added C24: 10u, Capacitor_SMD:C_0805_2012Metric, F.Cu at (184.6, 72.7)
- added C25: 1u, Capacitor_SMD:C_0603_1608Metric_Pad1.08x0.95mm_HandSolder, F.Cu at (166.2, 94.6)
- added C26: 100n, Capacitor_SMD:C_0603_1608Metric_Pad1.08x0.95mm_HandSolder, F.Cu at (165.6, 98.6)
- added C27: 100n, Capacitor_SMD:C_0603_1608Metric_Pad1.08x0.95mm_HandSolder, F.Cu at (154.6, 98.6)
- added C28: 10n, Capacitor_SMD:C_0603_1608Metric_Pad1.08x0.95mm_HandSolder, F.Cu at (167.8, 98.6)
- added C29: 10n, Capacitor_SMD:C_0603_1608Metric_Pad1.08x0.95mm_HandSolder, F.Cu at (156.8, 98.6)
- added C3: 0.1u, Capacitor_SMD:C_0603_1608Metric_Pad1.08x0.95mm_HandSolder, F.Cu at (167.9, 86.2)
- added C30: 10n, Capacitor_SMD:C_0603_1608Metric_Pad1.08x0.95mm_HandSolder, F.Cu at (163.4, 98.6)
- added C31: 10n, Capacitor_SMD:C_0603_1608Metric_Pad1.08x0.95mm_HandSolder, F.Cu at (152.4, 98.6)
- added C4: 10u, Capacitor_SMD:C_0805_2012Metric, F.Cu at (171.4, 86.1)
- added C40: 4.7u, Capacitor_SMD:C_0805_2012Metric_Pad1.18x1.45mm_HandSolder, F.Cu at (157.5, 62.5)
- added C41: 100n, Capacitor_SMD:C_0603_1608Metric_Pad1.08x0.95mm_HandSolder, F.Cu at (157.6, 59.3)
- added C42: 100n, Capacitor_SMD:C_0603_1608Metric, F.Cu at (159.0, 53.1)
- added C43: 22u, Capacitor_SMD:C_1210_3225Metric_Pad1.33x2.70mm_HandSolder, F.Cu at (170.7, 47.3)
- added C44: 22u, Capacitor_SMD:C_1210_3225Metric_Pad1.33x2.70mm_HandSolder, F.Cu at (174.2, 47.3)
- added C45: 3.3u, Capacitor_SMD:C_0805_2012Metric_Pad1.18x1.45mm_HandSolder, F.Cu at (172.4, 58.4)
- added C46: 10u, Capacitor_SMD:C_0805_2012Metric_Pad1.18x1.45mm_HandSolder, F.Cu at (174.9, 63.8)
- added C47: 10u, Capacitor_SMD:C_0805_2012Metric_Pad1.18x1.45mm_HandSolder, F.Cu at (174.9, 67.4)
- added C48: 0.1u, Capacitor_SMD:C_0603_1608Metric_Pad1.08x0.95mm_HandSolder, F.Cu at (153.5, 42.4)
- added C49: 1u, Capacitor_SMD:C_0603_1608Metric_Pad1.08x0.95mm_HandSolder, F.Cu at (153.4, 48.9)
- added C5: 0.1u, Capacitor_SMD:C_0603_1608Metric_Pad1.08x0.95mm_HandSolder, F.Cu at (159.2, 84.2)
- added C50: 220n, Capacitor_SMD:C_0603_1608Metric_Pad1.08x0.95mm_HandSolder, F.Cu at (159.2, 46.3)
- added C51: 10n, Capacitor_SMD:C_0603_1608Metric_Pad1.08x0.95mm_HandSolder, F.Cu at (153.9, 54.4)
- added C52: 10u, Capacitor_SMD:C_0805_2012Metric_Pad1.18x1.45mm_HandSolder, F.Cu at (153.6, 59.0)
- added C53: 0.1u, Capacitor_SMD:C_0603_1608Metric_Pad1.08x0.95mm_HandSolder, F.Cu at (167.8, 39.2)
- added C54: 0.1u, Capacitor_SMD:C_0603_1608Metric_Pad1.08x0.95mm_HandSolder, F.Cu at (161.9, 39.2)
- added C55: 0.1u, Capacitor_SMD:C_0603_1608Metric_Pad1.08x0.95mm_HandSolder, F.Cu at (176.3, 53.7)
- added C56: 0.1u, Capacitor_SMD:C_0603_1608Metric_Pad1.08x0.95mm_HandSolder, F.Cu at (180.3, 51.9)
- added C57: 0.1u, Capacitor_SMD:C_0603_1608Metric_Pad1.08x0.95mm_HandSolder, F.Cu at (180.2, 56.8)
- added C58: 0.1u, Capacitor_SMD:C_0603_1608Metric_Pad1.08x0.95mm_HandSolder, F.Cu at (177.5, 56.4)
- added C59: 10u, Capacitor_SMD:C_0603_1608Metric_Pad1.08x0.95mm_HandSolder, F.Cu at (167.0, 91.5)
- added C6: 0.1u, Capacitor_SMD:C_0603_1608Metric_Pad1.08x0.95mm_HandSolder, F.Cu at (171.8, 67.1)
- added C7: 0.1u, Capacitor_SMD:C_0603_1608Metric_Pad1.08x0.95mm_HandSolder, F.Cu at (166.2, 86.2)
- added C8: 0.1u, Capacitor_SMD:C_0603_1608Metric_Pad1.08x0.95mm_HandSolder, F.Cu at (169.5, 86.2)
- added C9: 1u, Capacitor_SMD:C_0603_1608Metric_Pad1.08x0.95mm_HandSolder, F.Cu at (167.0, 89.9)
- added D1: RGB_LED, LHRS_Special:RGB_LED, F.Cu at (161.6, 85.9)
- added D10: SBA130CH-AU_R1_000A1, Diode_SMD:D_SOD-323_HandSoldering, F.Cu at (175.9, 60.2)
- added D11: SMBJ15CA, Diode_SMD:D_SMB, F.Cu at (165.0, 46.0)
- added D12: SMAF4758A, LHRS_Passives:SODFL5026X125N, F.Cu at (155.0, 46.2)
- added D13: LED, LED_SMD:LED_0603_1608Metric, F.Cu at (177.8, 76.7)
- added D14: LED, LED_SMD:LED_0603_1608Metric, F.Cu at (147.6, 66.0)
- added D15: LED, LED_SMD:LED_0603_1608Metric, F.Cu at (147.6, 68.4)
- added D2: TVS, Diode_SMD:D_SOD-323, F.Cu at (145.4, 85.3)
- added D3: LED, LED_SMD:LED_0603_1608Metric, F.Cu at (141.0, 85.3)
- added D4: CDSOT23-T24CAN, LHRS_Passives:CDSOT23-T24CAN, F.Cu at (178.5, 90.7)
- added D5: D5V0P4UR6SO-7, LHRS_ICs:D5V0P4UR6SO-7, F.Cu at (144.4, 101.6)
- added D7: D_Schottky, Diode_SMD:D_SOD-123, F.Cu at (186.9, 71.8)
- added D8: TPD2EUSB30DRTR, LHRS_ICs:TPD2EUSB30DRTR, F.Cu at (184.5, 75.3)
- added D9: D5V0P4UR6SO-7, LHRS_ICs:D5V0P4UR6SO-7, F.Cu at (159.9, 98.6)
- added F2: Fuse, LHRS_Power:Fuse-3557-2, F.Cu at (141.2, 50.3)
- added FB1: FerriteBead, Capacitor_SMD:C_0603_1608Metric_Pad1.08x0.95mm_HandSolder, F.Cu at (164.2, 86.5)
- added FB2: FerriteBead, Capacitor_SMD:C_0603_1608Metric_Pad1.08x0.95mm_HandSolder, F.Cu at (173.5, 86.9)
- added IC1: TCAN3413DR, LHRS_Passives:TCAN3413DR, F.Cu at (178.5, 85.0)
- added IC3: LM74502DDFR, LHRS_Power:LM74502DDFR, F.Cu at (155.1, 51.8)
- added J1: SWD_Header, LHRS_Connectors:SWD_Conn, F.Cu at (165.7, 66.4)
- added J11: CAN_OUT, LHRS_Connectors:Molex_Nano-Fit_105309-xx05_1x05_P2.50mm_Vertical, F.Cu at (179.2, 111.3)
- added J2: SWD, Connector_PinHeader_2.54mm:PinHeader_1x04_P2.54mm_Vertical, F.Cu at (179.8, 71.8)
- added J3: USB_C_Receptacle_USB2.0_16P, LHRS_Connectors:USB_C_Receptacle_GCT_USB4105-xx-A_16P_TopMnt_Horizontal, F.Cu at (188.2, 81.4)
- added J4: Nano-Fit 1x5, Connector_Molex:Molex_Nano-Fit_105313-xx05_1x05_P2.50mm_Horizontal, F.Cu at (149.4, 105.6)
- added J5: TC K-type, LHRS_Connectors:105313-2102, F.Cu at (166.0, 105.6)
- added J6: CAN_DEBUG, Connector_Molex:Molex_Nano-Fit_105309-xx04_1x04_P2.50mm_Vertical, F.Cu at (189.2, 99.3)
- added J7: CAN_IN, LHRS_Connectors:Molex_Nano-Fit_105309-xx05_1x05_P2.50mm_Vertical, F.Cu at (179.2, 103.9)
- added J8: TC K-type, LHRS_Connectors:105313-2102, F.Cu at (156.5, 105.6)
- added JP1: TRM, Connector_PinHeader_2.54mm:PinHeader_1x02_P2.54mm_Vertical, F.Cu at (175.0, 98.3)
- added JP3: SolderJumper_2_Open, Jumper:SolderJumper-2_P1.3mm_Open_RoundedPad1.0x1.5mm, F.Cu at (148.8, 57.5)
- added L2: 8.2u, LHRS_Passives:74439369082, F.Cu at (165.5, 56.3)
- added Q3: PSMN012-100YS, Package_TO_SOT_SMD:LFPAK56, F.Cu at (148.3, 44.6)
- added Q4: PSMN012-100YS, Package_TO_SOT_SMD:LFPAK56, F.Cu at (148.2, 52.0)
- added R1: 1k, Resistor_SMD:R_0603_1608Metric_Pad0.98x0.95mm_HandSolder, F.Cu at (162.5, 89.3)
- added R10: 60, Resistor_SMD:R_0603_1608Metric_Pad0.98x0.95mm_HandSolder, F.Cu at (175.0, 94.6)
- added R11: 5.1k, Resistor_SMD:R_0603_1608Metric_Pad0.98x0.95mm_HandSolder, F.Cu at (182.6, 84.0)
- added R12: 5.1k, Resistor_SMD:R_0603_1608Metric_Pad0.98x0.95mm_HandSolder, F.Cu at (189.1, 74.2)
- added R2: 10k, Resistor_SMD:R_0603_1608Metric_Pad0.98x0.95mm_HandSolder, F.Cu at (154.0, 80.3)
- added R21: 10k, Resistor_SMD:R_0603_1608Metric_Pad0.98x0.95mm_HandSolder, F.Cu at (153.3, 94.1)
- added R22: 100k, Resistor_SMD:R_0603_1608Metric, F.Cu at (172.2, 51.5)
- added R23: 19.1k, Resistor_SMD:R_0603_1608Metric, F.Cu at (172.2, 54.7)
- added R24: 10k, Resistor_SMD:R_0603_1608Metric_Pad0.98x0.95mm_HandSolder, F.Cu at (157.1, 42.4)
- added R25: 33, Resistor_SMD:R_0603_1608Metric_Pad0.98x0.95mm_HandSolder, F.Cu at (152.0, 51.6)
- added R26: 100k, Resistor_SMD:R_0603_1608Metric_Pad0.98x0.95mm_HandSolder, F.Cu at (167.1, 41.8)
- added R27: 7.32k, Resistor_SMD:R_0603_1608Metric_Pad0.98x0.95mm_HandSolder, F.Cu at (168.8, 41.8)
- added R28: 100k, Resistor_SMD:R_0603_1608Metric_Pad0.98x0.95mm_HandSolder, F.Cu at (161.1, 41.8)
- added R29: 1k, Resistor_SMD:R_0603_1608Metric_Pad0.98x0.95mm_HandSolder, F.Cu at (174.6, 76.7)
- added R3: 1k, Resistor_SMD:R_0603_1608Metric_Pad0.98x0.95mm_HandSolder, F.Cu at (160.9, 89.3)
- added R30: 1k, Resistor_SMD:R_0603_1608Metric_Pad0.98x0.95mm_HandSolder, F.Cu at (144.0, 66.0)
- added R31: 1k, Resistor_SMD:R_0603_1608Metric_Pad0.98x0.95mm_HandSolder, F.Cu at (144.0, 68.4)
- added R32: 15.8k, Resistor_SMD:R_0603_1608Metric_Pad0.98x0.95mm_HandSolder, F.Cu at (162.8, 41.8)
- added R33: 10k, Resistor_SMD:R_0603_1608Metric_Pad0.98x0.95mm_HandSolder, F.Cu at (182.7, 54.4)
- added R34: 1M, Resistor_SMD:R_0603_1608Metric_Pad0.98x0.95mm_HandSolder, F.Cu at (168.3, 102.3)
- added R35: 1M, Resistor_SMD:R_0603_1608Metric_Pad0.98x0.95mm_HandSolder, F.Cu at (158.7, 102.3)
- added R36: 1M, Resistor_SMD:R_0603_1608Metric_Pad0.98x0.95mm_HandSolder, F.Cu at (161.2, 102.3)
- added R37: 1M, Resistor_SMD:R_0603_1608Metric_Pad0.98x0.95mm_HandSolder, F.Cu at (151.5, 102.3)
- added R38: 1k, Resistor_SMD:R_0603_1608Metric_Pad0.98x0.95mm_HandSolder, F.Cu at (166.0, 102.3)
- added R39: 1k, Resistor_SMD:R_0603_1608Metric_Pad0.98x0.95mm_HandSolder, F.Cu at (156.5, 102.3)
- added R4: 1k, Resistor_SMD:R_0603_1608Metric_Pad0.98x0.95mm_HandSolder, F.Cu at (159.3, 89.3)
- added R40: 1k, Resistor_SMD:R_0603_1608Metric_Pad0.98x0.95mm_HandSolder, F.Cu at (163.5, 102.3)
- added R41: 22, Resistor_SMD:R_0603_1608Metric_Pad0.98x0.95mm_HandSolder, F.Cu at (157.5, 91.0)
- added R42: 22, Resistor_SMD:R_0603_1608Metric_Pad0.98x0.95mm_HandSolder, F.Cu at (164.3, 91.1)
- added R43: 1k, Resistor_SMD:R_0603_1608Metric_Pad0.98x0.95mm_HandSolder, F.Cu at (154.0, 102.3)
- added R48: 22, Resistor_SMD:R_0603_1608Metric_Pad0.98x0.95mm_HandSolder, F.Cu at (155.8, 91.0)
- added R5: 22, Resistor_SMD:R_0603_1608Metric_Pad0.98x0.95mm_HandSolder, F.Cu at (169.2, 71.8)
- added R6: 22, Resistor_SMD:R_0603_1608Metric_Pad0.98x0.95mm_HandSolder, F.Cu at (174.4, 69.3)
- added R60: 0, Resistor_SMD:R_0603_1608Metric_Pad0.98x0.95mm_HandSolder, F.Cu at (173.8, 103.9)
- added R61: 0, Resistor_SMD:R_0603_1608Metric_Pad0.98x0.95mm_HandSolder, F.Cu at (173.8, 111.3)
- added R66: 16k, Resistor_SMD:R_0603_1608Metric_Pad0.98x0.95mm_HandSolder, F.Cu at (176.3, 51.9)
- added R67: 4.7k, Resistor_SMD:R_0603_1608Metric_Pad0.98x0.95mm_HandSolder, F.Cu at (180.1, 58.9)
- added R7: 10k, Resistor_SMD:R_0603_1608Metric_Pad0.98x0.95mm_HandSolder, F.Cu at (151.6, 66.0)
- added R8: 1k, Resistor_SMD:R_0603_1608Metric_Pad0.98x0.95mm_HandSolder, F.Cu at (143.2, 85.3)
- added R9: 60, Resistor_SMD:R_0603_1608Metric_Pad0.98x0.95mm_HandSolder, F.Cu at (177.5, 93.4)
- added SW1: Reset, LHRS_Special:TL3365AF180QG, F.Cu at (154.6, 85.0)
- added SW2: SW_SPDT, LHRS_Special:BootSW, F.Cu at (144.3, 77.5)
- added TP10: TCN, TestPoint:TestPoint_Pad_D1.5mm, F.Cu at (170.6, 102.8)
- added TP11: TCN, TestPoint:TestPoint_Pad_D1.5mm, F.Cu at (150.1, 96.4)
- added TP2: SDA, TestPoint:TestPoint_Pad_D1.5mm, F.Cu at (148.4, 101.9)
- added TP3: SCL, TestPoint:TestPoint_Pad_D1.5mm, F.Cu at (140.6, 100.4)
- added TP38: +12V, TestPoint:TestPoint_Pad_D1.5mm, F.Cu at (139.9, 62.1)
- added TP39: +12V_PP, TestPoint:TestPoint_Pad_D1.5mm, F.Cu at (146.5, 62.9)
- added TP40: +5V_BUCK, TestPoint:TestPoint_Pad_D1.5mm, F.Cu at (189.5, 40.0)
- added TP41: +USBC_5V, TestPoint:TestPoint_Pad_D1.5mm, F.Cu at (189.8, 66.0)
- added TP42: MUX_OUT, TestPoint:TestPoint_Pad_D1.5mm, F.Cu at (189.5, 44.0)
- added TP43: LDO_OUT_TestPoint, TestPoint:TestPoint_Pad_D1.5mm, F.Cu at (189.5, 48.0)
- added TP44: Power TestPoint, TestPoint:TestPoint_Pad_D1.5mm, F.Cu at (189.5, 52.0)
- added TP45: MCU TestPoint, TestPoint:TestPoint_Pad_D1.5mm, F.Cu at (173.4, 109.0)
- added TP46: CAN TestPoint, TestPoint:TestPoint_Pad_D1.5mm, F.Cu at (173.2, 106.2)
- added TP47: SPI_MISO, TestPoint:TestPoint_Pad_D1.5mm, F.Cu at (170.3, 105.7)
- added TP48: SPI_MOSI, TestPoint:TestPoint_Pad_D1.5mm, F.Cu at (170.3, 108.5)
- added TP49: SPI_SCK, TestPoint:TestPoint_Pad_D1.5mm, F.Cu at (170.6, 111.2)
- added TP5: V_in_12V, Connector_PinHeader_2.54mm:PinHeader_1x01_P2.54mm_Vertical, F.Cu at (143.3, 62.6)
- added TP6: TC_ADC_CS, TestPoint:TestPoint_Pad_D1.5mm, F.Cu at (150.1, 93.6)
- added TP7: TCP, TestPoint:TestPoint_Pad_D1.5mm, F.Cu at (173.8, 101.7)
- added TP8: TCP, TestPoint:TestPoint_Pad_D1.5mm, F.Cu at (150.1, 99.2)
- added TP_3.3V2: 3.3V, TestPoint:TestPoint_Loop_D1.80mm_Drill1.0mm_Beaded, F.Cu at (178.8, 46.0)
- added U1: STM32G473CETx, LHRS_Special:48PinMCU, F.Cu at (167.0, 79.0)
- added U3: ADS1118IDGS, Package_SO:TSSOP-10_3x3mm_P0.5mm, F.Cu at (159.9, 94.6)
- added U5: LMR51635XDDCR, LHRS_ICs:DDC0006A-MFG, F.Cu at (157.8, 56.6)
- added U6: MCP1826S, Package_TO_SOT_SMD:SOT-223-3_TabPin2, F.Cu at (181.6, 64.7)
- added U7: TPS2117DRLR, LHRS_Power:TPS2117DRLR, F.Cu at (180.5, 54.3)
- added Y1: Crystal, LHRS_Passives:Crystal_SMD_Abracon_ABM3-2Pin_5.0x3.2mm, F.Cu at (158.4, 78.8)
Other:
- board outline added: 56.3 x 82.6 mm
- copper layers 0 -> 2
- board text added: "+"
- board text added: "-"
- board text added: "12V"
- board text added: "3V3"
- board text added: "CH"
- board text added: "CL"
- board text added: "CLK"
- board text added: "DIO"
- board text added: "GND"
- board text added: "NC"
- board text added: "SCL"
- board text added: "SDA"
- board text added: "SH"
- board text added: "TC0"
- board text added: "TC1"
