File: hardware/TC_Channel.kicad_sch (KiCad schematic)
At the start: 0 parts

Commit message: irradescence stuff
Parts:
- added C27: 100n, Capacitor_SMD:C_0603_1608Metric_Pad1.08x0.95mm_HandSolder, symbol Device:C
- added C29, C31: 10n, Capacitor_SMD:C_0603_1608Metric_Pad1.08x0.95mm_HandSolder, symbol Device:C
- added D9: TPD2EUSB30DRTR, LHRS_ICs:TPD2EUSB30DRTR, symbol lhrs_ics:TPD2EUSB30DRTR
- added J8: TC K-type, LHRS_Connectors:105313-2102, symbol Connector_Generic:Conn_01x02
- added R35, R37: 1M, Resistor_SMD:R_0603_1608Metric_Pad0.98x0.95mm_HandSolder, symbol Device:R
- added R39, R43: 1k, Resistor_SMD:R_0603_1608Metric_Pad0.98x0.95mm_HandSolder, symbol Device:R
- added TP11: TCN, TestPoint:TestPoint_Pad_D1.5mm, symbol Connector:TestPoint
- added TP8: TCP, TestPoint:TestPoint_Pad_D1.5mm, symbol Connector:TestPoint
Connections:
- net +3.3V: now also R35.1
- net GND: now also C29.2, C31.2, D9.3 (GND), R37.2
- net TCN: now also C27.2, C31.1, R43.2, TP11.1
- net TCP: now also C27.1, C29.1, R39.2, TP8.1
- new net TC_N: D9.2 (D-), J8.2 (Pin_2), R37.1, R43.1
- new net TC_P: D9.1 (D+), J8.1 (Pin_1), R35.2, R39.1
Other:
- note added: "ESD"
- note added: "Test Points"
- note removed: "1M from TC+ to +3.3V 1M from TC- to GND Sets common mode near mid-supply and drives the reading to +FS if the thermocouple is unplugged/open."
- note removed: "ESD + Test Points"
- note removed: "J?: K-type TC input. Options: - Mini K-type socket (yellow, Omega PCC-SMP-K style) - or 2-pin Nano-Fit if the harness lead prefers Label pins TC+ (yellow tape lead) / TC-. Copper between connector and ADC = cold junction; keep both TC traces symmetric."
- note removed: "Open-TC Bias"
- note removed: "Series 1k on each line, 100 nF differential (TC+ to TC-), 10 nF each line to GND (common mode). Write the cutoffs on the sheet (review comment from strain gauge)."
- note removed: "TPD2EUSB30 on TC+/TC-, pin 3 -> GND, at the connector. TP on TCP and TCN."
- company: Longhorn Racing Solar - VCAT Telemetry -> (none)
- title: Thermocouple Input Channel -> (none)

Commit message: check breakout board layout
Parts:
- removed D9: TPD2EUSB30DRTR, LHRS_ICs:TPD2EUSB30DRTR, symbol lhrs_ics:TPD2EUSB30DRTR
Other:
- note removed: "ESD"
Changed lines of the file:
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@@
-	)
-	(rectangle
-		(start 46.99 25.4)
-		(end 92.71 40.64)
-		(stroke
-			(width 0)
-			(type default)
-		)
-		(fill
-			(type none)
-		)
 	)
 	(rectangle
@@
 		(exclude_from_sim no)
 		(at 95.25 24.13 0)
-		(effects
-			(font
-				(size 1.27 1.27)
-			)
-			(justify left)
-		)
-	)
-	(text "ESD"
-		(exclude_from_sim no)
-		(at 46.99 24.13 0)
 		(effects
 			(font
@@
 	(wire
 		(pts
-			(xy 82.55 33.02) (xy 85.09 33.02)
-		)
-		(stroke
-			(width 0)
-			(type default)
-		)
-	)
-	(wire
-		(pts
 			(xy 68.58 68.58) (xy 71.12 68.58)
 		)
@@
 	(wire
 		(pts
+			(xy 35.56 93.98) (xy 34.29 93.98)
+		)
+		(stroke
+			(width 0)
+			(type default)
+		)
+	)
+	(wire
+		(pts
 			(xy 30.48 34.29) (xy 33.02 34.29)
 		)
@@
 	(wire
 		(pts
-			(xy 34.29 91.44) (xy 34.29 93.98)
-		)
-		(stroke
-			(width 0)
-			(type default)
-		)
-	)
-	(wire
-		(pts
 			(xy 68.58 71.12) (xy 68.58 68.58)
 		)
@@
 	(wire
 		(pts
+			(xy 34.29 93.98) (xy 34.29 91.44)
+		)
+		(stroke
+			(width 0)
+			(type default)
+		)
+	)
+	(wire
+		(pts
 			(xy 34.29 66.04) (xy 34.29 68.58)
 		)
@@
 	(wire
 		(pts
-			(xy 57.15 33.02) (xy 54.61 33.02)
-		)
-		(stroke
-			(width 0)
-			(type default)
-		)
-	)
-	(wire
-		(pts
 			(xy 55.88 91.44) (xy 55.88 90.17)
 		)
@@
 	(wire
 		(pts
-			(xy 57.15 35.56) (xy 54.61 35.56)
-		)
-		(stroke
-			(width 0)
-			(type default)
-		)
-	)
-	(wire
-		(pts
 			(xy 36.83 81.28) (xy 34.29 81.28)
 		)
@@
 		)
 	)
-	(label "TC_P"
+	(hierarchical_label "TC_P"
+		(shape passive)
 		(at 33.02 31.75 0)
 		(effects
@@
 				(size 1.27 1.27)
 			)
-			(justify left bottom)
-		)
-	)
-	(label "TC_P"
+			(justify left)
+		)
+	)
+	(hierarchical_label "TC_P"
+		(shape passive)
 		(at 29.21 68.58 180)
 		(effects
@@
 				(size 1.27 1.27)
 			)
-			(justify right bottom)
-		)
-	)
-	(label "TC_N"
+			(justify right)
+		)
+	)
+	(hierarchical_label "TC_N"
+		(shape passive)
 		(at 29.21 81.28 180)
 		(effects
@@
 				(size 1.27 1.27)
 			)
-			(justify right bottom)
-		)
-	)
-	(label "TC_N"
-		(at 54.61 35.56 180)
-		(effects
-			(font
-				(size 1.27 1.27)
-			)
-			(justify right bottom)
-		)
-	)
-	(label "TC_P"
-		(at 54.61 33.02 180)
-		(effects
-			(font
-				(size 1.27 1.27)
-			)
-			(justify right bottom)
-		)
-	)
-	(label "TC_N"
+			(justify right)
+		)
+	)
+	(hierarchical_label "TC_N"
+		(shape passive)
 		(at 33.02 34.29 0)
 		(effects
@@
 				(size 1.27 1.27)
 			)
-			(justify left bottom)
+			(justify left)
 		)
 	)
 	(hierarchical_label "GND"
 		(shape passive)
-		(at 34.29 93.98 270)
-		(effects
-			(font
-				(size 1.27 1.27)
-			)
-			(justify right)
+		(at 35.56 93.98 0)
+		(effects
+			(font
+				(size 1.27 1.27)
+			)
+			(justify left)
 		)
 	)
@@
 		(shape output)
 		(at 71.12 68.58 0)
-		(effects
-			(font
-				(size 1.27 1.27)
-			)
-			(justify left)
-		)
-	)
-	(hierarchical_label "GND"
-		(shape passive)
-		(at 85.09 33.02 0)
 		(effects
 			(font
@@
 					(unit 1)
 				)
-			)
-		)
-	)
-	(symbol
-		(lib_id "lhrs_ics:TPD2EUSB30DRTR")
-		(at 57.15 33.02 0)
-		(unit 1)
-		(body_style 1)
-		(exclude_from_sim no)
-		(in_bom yes)
-		(on_board yes)
-		(in_pos_files yes)
-		(dnp no)
-		(property "Reference" "D9"
-			(at 69.85 39.624 0)
-			(show_name no)
-			(do_not_autoplace no)
-			(effects
-				(font
-					(size 1.27 1.27)
-				)
-			)
-		)
-		(property "Value" "TPD2EUSB30DRTR"
-			(at 69.85 27.94 0)
-			(show_name no)
-			(do_not_autoplace no)
-			(effects
-				(font
-					(size 1.27 1.27)
-				)
-			)
-		)
-		(property "Footprint" "LHRS_ICs:TPD2EUSB30DRTR"
-			(at 57.15 33.02 0)
-			(hide yes)
-			(show_name no)
-			(do_not_autoplace no)
-			(effects
-				(font
-					(size 1.27 1.27)
-				)
-			)
-		)
-		(property "Datasheet" "~"
-			(at 57.15 33.02 0)
-			(hide yes)
-			(show_name no)
-			(do_not_autoplace no)
-			(effects
-				(font
-					(size 1.27 1.27)
-				)
-			)
-		)
-		(property "Description" ""
-			(at 57.15 33.02 0)
-			(hide yes)
-			(show_name no)
-			(do_not_autoplace no)
-			(effects
-				(font
-					(size 1.27 1.27)
-				)
-			)
-		)
-		(pin "1"
-		)
-		(pin "2"
-		)
-		(pin "3"
-		)
-		(instances
-			(project "BlackBodyBoard"
-				(path "/48096f47-ddef-4ea4-8e15-14613f1872f0/59189416-5d51-4d24-8c42-809517448b9b/640f9422-f4a8-43eb-92f9-235dd3a04ddb"
-					(reference "D6")
-					(unit 1)
-				)
-				(path "/48096f47-ddef-4ea4-8e15-14613f1872f0/59189416-5d51-4d24-8c42-809517448b9b/dedb1a1b-2ed4-4982-a0d7-8b88c87cf280"
-					(reference "D9")
-					(unit 1)
-				)

Commit message: Main board placement + silkscreen, breakout ground plane, DRC rule updates
- Grouped placement and condensed outline (2 mm rounded corners)
- Silkscreen refs moved next to their parts, pin labels added
- Interrupt removed from main board and breakout (test point instead)
- Breakout: B.Cu ground plane + stitching vias
- Default clearance / hole clearance lowered to 0.15 mm
Parts:
- C27: LCSC P/N (none) -> C1591; P/N (none) -> CL10B104KB8NNNC
- C29, C31: LCSC P/N (none) -> C100042; P/N (none) -> CC0603KRX7R9BB103
- J8: P/N (none) -> 1053132102
- R35, R37: LCSC P/N (none) -> C22935; P/N (none) -> 0603WAF1004T5E
- R39, R43: LCSC P/N (none) -> C21190; P/N (none) -> 0603WAF1001T5E
Changed lines of the file:
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@@
+		)
+	)
+	(hierarchical_label "GND"
+		(shape passive)
+		(at 35.56 93.98 0)
+		(effects
+			(font
+				(size 1.27 1.27)
+			)
+			(justify left)
+		)
+	)
+	(hierarchical_label "TCP"
+		(shape output)
+		(at 107.95 34.29 0)
+		(effects
+			(font
+				(size 1.27 1.27)
+			)
+			(justify left)
+		)
+	)
+	(hierarchical_label "TCP"
+		(shape output)
+		(at 71.12 68.58 0)
+		(effects
+			(font
+				(size 1.27 1.27)
+			)
+			(justify left)
 		)
 	)
@@
 		)
 	)
-	(hierarchical_label "TC_N"
-		(shape passive)
-		(at 33.02 34.29 0)
-		(effects
-			(font
-				(size 1.27 1.27)
-			)
-			(justify left)
-		)
-	)
-	(hierarchical_label "GND"
-		(shape passive)
-		(at 35.56 93.98 0)
-		(effects
-			(font
-				(size 1.27 1.27)
-			)
-			(justify left)
-		)
-	)
-	(hierarchical_label "TCP"
-		(shape output)
-		(at 107.95 34.29 0)
-		(effects
-			(font
-				(size 1.27 1.27)
-			)
-			(justify left)
-		)
-	)
-	(hierarchical_label "TCP"
-		(shape output)
-		(at 71.12 68.58 0)
-		(effects
-			(font
-				(size 1.27 1.27)
-			)
-			(justify left)
-		)
-	)
 	(hierarchical_label "GND"
 		(shape passive)
@@
 		(shape output)
 		(at 125.73 34.29 0)
+		(effects
+			(font
+				(size 1.27 1.27)
+			)
+			(justify left)
+		)
+	)
+	(hierarchical_label "TC_N"
+		(shape passive)
+		(at 33.02 34.29 0)
 		(effects
 			(font
@@
 			)
 		)
+		(property "P/N" "CC0603KRX7R9BB103"
+			(at 55.88 73.66 0)
+			(hide yes)
+			(show_name no)
+			(do_not_autoplace no)
+			(effects
+				(font
+					(size 1.27 1.27)
+				)
+			)
+		)
+		(property "LCSC P/N" "C100042"
+			(at 55.88 73.66 0)
+			(hide yes)
+			(show_name no)
+			(do_not_autoplace no)
+			(effects
+				(font
+					(size 1.27 1.27)
+				)
+			)
+		)
 		(pin "1"
 		)
@@
 			)
 		)
+		(property "P/N" "CC0603KRX7R9BB103"
+			(at 55.88 86.36 0)
+			(hide yes)
+			(show_name no)
+			(do_not_autoplace no)
+			(effects
+				(font
+					(size 1.27 1.27)
+				)
+			)
+		)
+		(property "LCSC P/N" "C100042"
+			(at 55.88 86.36 0)
+			(hide yes)
+			(show_name no)
+			(do_not_autoplace no)
+			(effects
+				(font
+					(size 1.27 1.27)
+				)
+			)
+		)
 		(pin "1"
 		)
@@
 		)
 		(property "Description" ""
+			(at 68.58 74.93 0)
+			(hide yes)
+			(show_name no)
+			(do_not_autoplace no)
+			(effects
+				(font
+					(size 1.27 1.27)
+				)
+			)
+		)
+		(property "P/N" "CL10B104KB8NNNC"
+			(at 68.58 74.93 0)
+			(hide yes)
+			(show_name no)
+			(do_not_autoplace no)
+			(effects
+				(font
+					(size 1.27 1.27)
+				)
+			)
+		)
+		(property "LCSC P/N" "C1591"
 			(at 68.58 74.93 0)
 			(hide yes)
@@
 			)
 		)
+		(property "P/N" "1053132102"
+			(at 25.4 31.75 0)
+			(hide yes)
+			(show_name no)
+			(do_not_autoplace no)
+			(effects
+				(font
+					(size 1.27 1.27)
+				)
+			)
+		)
 		(pin "1"
 		)
@@
 			)
 		)
+		(property "P/N" "0603WAF1004T5E"
+			(at 34.29 87.63 0)
+			(hide yes)
+			(show_name no)
+			(do_not_autoplace no)
+			(effects
+				(font
+					(size 1.27 1.27)
+				)
+			)
+		)
+		(property "LCSC P/N" "C22935"
+			(at 34.29 87.63 0)
+			(hide yes)
+			(show_name no)
+			(do_not_autoplace no)
+			(effects
+				(font
+					(size 1.27 1.27)
+				)
+			)
+		)
 		(pin "1"
 		)
@@
 			)
 		)
+		(property "P/N" "0603WAF1001T5E"
+			(at 40.64 68.58 0)
+			(hide yes)
+			(show_name no)
+			(do_not_autoplace no)
+			(effects
+				(font
+					(size 1.27 1.27)
+				)
+			)
+		)
+		(property "LCSC P/N" "C21190"
+			(at 40.64 68.58 0)
+			(hide yes)
+			(show_name no)
+			(do_not_autoplace no)
+			(effects
+				(font
+					(size 1.27 1.27)
+				)
+			)
+		)
 		(pin "1"
 		)
@@
 			)
 		)
+		(property "P/N" "0603WAF1004T5E"
+			(at 34.29 62.23 0)
+			(hide yes)
+			(show_name no)
+			(do_not_autoplace no)
+			(effects
+				(font
+					(size 1.27 1.27)
+				)
+			)
+		)
+		(property "LCSC P/N" "C22935"
+			(at 34.29 62.23 0)
+			(hide yes)
+			(show_name no)
+			(do_not_autoplace no)
+			(effects
+				(font
+					(size 1.27 1.27)
+				)
+			)
+		)
 		(pin "1"
 		)
@@
 			(at 40.64 81.28 0)
 			(hide yes)
+			(show_name no)
+			(do_not_autoplace no)
+			(effects
+				(font
+					(size 1.27 1.27)
+				)
+			)
+		)
+		(property "P/N" "0603WAF1001T5E"
+			(at 40.64 81.28 0)
+			(hide yes)
+			(show_name no)
+			(do_not_autoplace no)
+			(effects
+				(font
+					(size 1.27 1.27)
+				)
+			)
+		)
+		(property "LCSC P/N" "C21190"
+			(at 40.64 81.28 0)
+			(hide yes)
