File: hardware/Thermocouple.kicad_sch (KiCad schematic)
At the start: 0 parts

Commit message: irradescence stuff
Parts:
- added C23: 0.1u, Capacitor_SMD:C_0603_1608Metric_Pad1.08x0.95mm_HandSolder, symbol Device:C
- added C25: 1u, Capacitor_SMD:C_0603_1608Metric_Pad1.08x0.95mm_HandSolder, symbol Device:C
- added R20: 22, Resistor_SMD:R_0603_1608Metric_Pad0.98x0.95mm_HandSolder, symbol Device:R
- added R21: 10k, Resistor_SMD:R_0603_1608Metric_Pad0.98x0.95mm_HandSolder, symbol Device:R
- added TP6: TC_ADC_CS, TestPoint:TestPoint_Pad_D1.5mm, symbol Connector:TestPoint
- added U3: ADS1118IDGS, Package_SO:VSSOP-10_3x3mm_P0.5mm, symbol BlackBody:ADS1118IDGS
Connections:
- net +3.3V: now also C23.1, C25.1, R21.1, U3.8 (VDD)
- net GND: now also C23.2, C25.2, U3.3 (GND)
- net SPI_MISO: now also R20.2
- net SPI_MOSI: now also U3.10 (DIN)
- net SPI_SCK: now also U3.1 (SCLK)
- net TC0N: now also U3.4 (AIN0)
- net TC0P: now also U3.5 (AIN1)
- net TC1N: now also U3.6 (AIN2)
- net TC1P: now also U3.7 (AIN3)
- net TC_ADC_CS: now also R21.2, TP6.1, U3.2 (~{CS})
- new net: R20.1, U3.9 (DOUT/~{DRDY})
Other:
- note added: "ADS1118"
- note added: "SPI test points + ESD are on the root sheet"
- note added: "Test Point"
- note removed: "ADS1118 (16-bit ADC + cold-junction sensor)"
- note removed: "Firmware Notes"
- note removed: "K-type: ~41 uV/C. T = NIST K-type inverse(V_tc + V(T_cj)). Use the NIST polynomial or a lookup table. Open TC: bias resistors in each channel pull the input to full scale -> reading pinned at +FS = 'TC open' fault. CAN: module temp at 2 Hz; validity bit per channel; board temp optional (from ADS1118 internal sensor)."
- note removed: "TP on SPI_SCK, SPI_MISO, SPI_MOSI, TC_ADC_CS. Add TPD2EUSB30 on the SPI test points (same as strain gauge: SCK+MOSI, MISO+CS)."
- note removed: "Test Points"
- note removed: "U?: ADS1118IDGSR (LCSC C55347, ~$1.75 @10). Replaces MCP96L00 (I2C, locked up until power-cycled). AIN0/AIN1 = TC0P/TC0N AIN2/AIN3 = TC1P/TC1N SCLK = SPI_SCK DIN = SPI_MOSI CS = TC_ADC_CS (10k pull-up to +3.3V) DOUT/DRDY = SPI_MISO (22R at the pin; DRDY is muxed on DOUT, no extra GPIO) VDD = +3.3V with 0.1 uF + 1 uF to GND. GND = GND. Settings: PGA +/-0.256 V, 128 SPS, alternate TC0 / TC1 / inter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"
- company: Longhorn Racing Solar - VCAT Telemetry -> (none)
- title: Thermocouple ADC -> (none)

Commit message: check breakout board layout
Parts:
- removed R20: 22, Resistor_SMD:R_0603_1608Metric_Pad0.98x0.95mm_HandSolder, symbol Device:R
- added D9: D5V0P4UR6SO-7, LHRS_ICs:D5V0P4UR6SO-7, symbol lhrs_ics:D5V0P4UR6SO-7
- U3: footprint Package_SO:VSSOP-10_3x3mm_P0.5mm -> Package_SO:TSSOP-10_3x3mm_P0.5mm
Connections:
- net +3.3V: now also D9.5
- net GND: now also D9.2
- net SPI_MISO: now also U3.9 (DOUT/~{DRDY})
- new net TC0+: D9.1
- new net TC0-: D9.3
- new net TC1+: D9.6
- new net TC1-: D9.4
Other:
- sheet TC_Channel0 ports: added TC_N, TC_P; removed none
- sheet TC_Channel1 ports: added TC_N, TC_P; removed none
- note added: "Thermocouple ESD"

Commit message: Main board placement + silkscreen, breakout ground plane, DRC rule updates
- Grouped placement and condensed outline (2 mm rounded corners)
- Silkscreen refs moved next to their parts, pin labels added
- Interrupt removed from main board and breakout (test point instead)
- Breakout: B.Cu ground plane + stitching vias
- Default clearance / hole clearance lowered to 0.15 mm
Parts:
- C23: value 0.1u -> 100n; LCSC P/N (none) -> C1591; P/N (none) -> CL10B104KB8NNNC
- C25: LCSC P/N (none) -> C15849; P/N (none) -> CC0603KRX7R9BB105
- R21: LCSC P/N (none) -> C25804; P/N (none) -> 0603WAF1002T5E
- U3: LCSC P/N (none) -> C55347; P/N (none) -> ADS1118IDGSR
