File: hardware/IrradianceBreakout/IrradianceBreakout.kicad_sch (KiCad schematic)
At the start: 0 parts

Commit message: irradescence stuff
Parts:
- added D1: BPW34, symbol BlackBody:BPW34
- added J1: Nano-Fit 1x5, Connector_Molex:Molex_Nano-Fit_105313-xx05_1x05_P2.50mm_Horizontal, symbol Connector_Generic:Conn_01x05
Connections:
- new net GNDA: J1.3 (Pin_3), J1.4 (Pin_4)
- new net PD_A: D1.1 (A), J1.2 (Pin_2)
- new net PD_K: D1.2 (K), J1.1 (Pin_1)
- no-connect marks 0 -> 1
Other:
- note added: "Same Nano-Fit 1x5 as the main board J. BRK_DET tied to GNDA here (main board reads low = present). Shield not connected here (terminated on the main board only)."
- note added: "Vishay BPW34 / BPW34S, 430-1100 nm, 7.5 mm2. Top side, centred on the window. Assign the footprint once the exact package is picked."
- note removed: "D?: Vishay BPW34 / BPW34S silicon PIN photodiode (430-1100 nm, peak ~900 nm, 7.5 mm2). Anode -> PD_A, Cathode -> PD_K. No bias, no local electronics: the TIA lives on the main Blackbody board (photovoltaic mode). Place on the TOP side, centered on the window. Optional: PTFE/opal diffuser over it for cosine response."
- note removed: "J?: same Nano-Fit series as the main board end. PD_A, PD_K (twisted pair), BRK_DET, GNDA, SHIELD. BRK_DET: tie to GNDA on THIS board so the main board can detect a missing/unplugged breakout. SHIELD: leave unconnected here (terminated at the main board only)."
- note removed: "Mechanical"
- note removed: "Mount on the underside of the top shell behind a window (Ravi); match the module tilt (Aarav). Keep the board tiny; 2 mounting holes. Old breakout: Power-Generation-Blackbody/ Hardware/IrradianceBreakout (TSL2591, I2C)."
- company: Longhorn Racing Solar - VCAT Telemetry -> (none)
- title: Blackbody Irradiance Breakout -> (none)
Changed lines of the file:
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@@
-(kicad_sch
-	(version 20260306)
-	(generator "eeschema")
-	(generator_version "10.0")
-	(paper "A4")
-	(title_block
-		(title "Blackbody Irradiance Breakout")
-		(rev "A")
-		(company "Longhorn Racing Solar - VCAT Telemetry")
-	)
-	(text "Photodiode"
-		(exclude_from_sim no)
-		(at 25.4 27.94 0)
-		(effects
-			(font
-				(size 1.27 1.27)
-				(bold yes)
-			)
-			(justify left top)
-		)
-	)
-	(rectangle
-		(start 25.4 30.48)
-		(end 101.6 76.2)
-		(stroke
-			(width 0)
-			(type default)
-		)
-		(fill
-			(type none)
-		)
-	)
-	(text "D?: Vishay BPW34 / BPW34S silicon PIN photodiode\n(430-1100 nm, peak ~900 nm, 7.5 mm2).\n\nAnode -> PD_A, Cathode -> PD_K.\nNo bias, no local electronics: the TIA lives on the\nmain Blackbody board (photovoltaic mode).\n\nPlace on the TOP side, centered on the window.\nOptional: PTFE/opal diffuser over it for cosine response."
-		(exclude_from_sim no)
-		(at 26.669999999999998 31.75 0)
-		(effects
-			(font
-				(size 1.27 1.27)
-			)
-			(justify left top)
-		)
-	)
-	(text "Harness Connector"
-		(exclude_from_sim no)
-		(at 106.68 27.94 0)
-		(effects
-			(font
-				(size 1.27 1.27)
-				(bold yes)
-			)
-			(justify left top)
-		)
-	)
-	(rectangle
-		(start 106.68 30.48)
-		(end 177.8 76.2)
-		(stroke
-			(width 0)
-			(type default)
-		)
-		(fill
-			(type none)
-		)
-	)
-	(text "J?: same Nano-Fit series as the main board end.\nPD_A, PD_K (twisted pair), BRK_DET, GNDA, SHIELD.\n\nBRK_DET: tie to GNDA on THIS board so the main\nboard can detect a missing/unplugged breakout.\nSHIELD: leave unconnected here (terminated at the\nmain board only)."
-		(exclude_from_sim no)
-		(at 107.95 31.75 0)
-		(effects
-			(font
-				(size 1.27 1.27)
-			)
-			(justify left top)
-		)
-	)
-	(text "Mechanical"
-		(exclude_from_sim no)
-		(at 182.88 27.94 0)
-		(effects
-			(font
-				(size 1.27 1.27)
-				(bold yes)
-			)
-			(justify left top)
-		)
-	)
-	(rectangle
-		(start 182.88 30.48)
-		(end 266.7 76.2)
-		(stroke
-			(width 0)
-			(type default)
-		)
-		(fill
-			(type none)
-		)
-	)
-	(text "Mount on the underside of the top shell behind a\nwindow (Ravi); match the module tilt (Aarav).\nKeep the board tiny; 2 mounting holes.\nOld breakout: Power-Generation-Blackbody/\nHardware/IrradianceBreakout (TSL2591, I2C)."
-		(exclude_from_sim no)
-		(at 184.15 31.75 0)
-		(effects
-			(font
-				(size 1.27 1.27)
-			)
-			(justify left top)
-		)
-	)
-	(sheet_instances
-		(path "/"
-			(page "1")
-		)
-	)
+(kicad_sch (version 20260306) (generator "eeschema") (generator_version "10.0") (paper "A4")
+	(text "Photodiode" (exclude_from_sim no) (at 20.32 24.13 0) (effects (font (size 1.27 1.27)) (justify left)))
+	(rectangle (start 20.32 25.4) (end 96.52 76.2) (stroke (width 0) (type default)) (fill (type none)))
+	(text "Vishay BPW34 / BPW34S, 430-1100 nm, 7.5 mm2. Top side, centred on the window.\nAssign the footprint once the exact package is picked." (exclude_from_sim no) (at 20.32 77.47 0) (effects (font (size 1.27 1.27)) (justify left top)))
+	(symbol (lib_id "BlackBody:BPW34") (at 53.34 45.72 0) (unit 1) (body_style 1) (exclude_from_sim no) (in_bom yes) (on_board yes) (in_pos_files yes) (dnp no) (fields_autoplaced no) (property "Reference" "D1" (at 53.34 49.53 0) (show_name no) (do_not_autoplace no) (effects (font (size 1.27 1.27)))) (property "Value" "BPW34" (at 53.34 41.91 0) (show_name no) (do_not_autoplace no) (effects (font (size 1.27 1.27)))) (property "Footprint" "" (at 53.34 45.72 0) (show_name no) (do_not_autoplace no) (hide yes) (effects (font (size 1.27 1.27)))) (property "Datasheet" "~" (at 53.34 45.72 0) (show_name no) (do_not_autoplace no) (hide yes) (effects (font (size 1.27 1.27)))) (property "Description" "" (at 53.34 45.72 0) (show_name no) (do_not_autoplace no) (hide yes) (effects (font (size 1.27 1.27)))) (pin "1") (pin "2") (instances (project "IrradianceBreakout" (path "/552486ca-d81b-4f74-b370-4ec84ac435dd" (reference "D1") (unit 1)))))
+	(wire (pts (xy 49.53 45.72) (xy 46.99 45.72)) (stroke (width 0) (type default)))
+	(label "PD_A" (at 46.99 45.72 180) (effects (font (size 1.27 1.27)) (justify right bottom)))
+	(wire (pts (xy 57.15 45.72) (xy 59.69 45.72)) (stroke (width 0) (type default)))
+	(label "PD_K" (at 59.69 45.72 0) (effects (font (size 1.27 1.27)) (justify left bottom)))
+	(text "Harness Connector" (exclude_from_sim no) (at 101.6 24.13 0) (effects (font (size 1.27 1.27)) (justify left)))
+	(rectangle (start 101.6 25.4) (end 177.8 76.2) (stroke (width 0) (type default)) (fill (type none)))
+	(text "Same Nano-Fit 1x5 as the main board J.\nBRK_DET tied to GNDA here (main board reads low = present).\nShield not connected here (terminated on the main board only)." (exclude_from_sim no) (at 101.6 77.47 0) (effects (font (size 1.27 1.27)) (justify left top)))
+	(symbol (lib_id "Connector_Generic:Conn_01x05") (at 139.7 45.72 0) (unit 1) (body_style 1) (exclude_from_sim no) (in_bom yes) (on_board yes) (in_pos_files yes) (dnp no) (fields_autoplaced no) (property "Reference" "J1" (at 137.16 36.83 0) (show_name no) (do_not_autoplace no) (effects (font (size 1.27 1.27)))) (property "Value" "Nano-Fit 1x5" (at 137.16 54.61 0) (show_name no) (do_not_autoplace no) (effects (font (size 1.27 1.27)))) (property "Footprint" "Connector_Molex:Molex_Nano-Fit_105313-xx05_1x05_P2.50mm_Horizontal" (at 139.7 45.72 0) (show_name no) (do_not_autoplace no) (hide yes) (effects (font (size 1.27 1.27)))) (property "Datasheet" "~" (at 139.7 45.72 0) (show_name no) (do_not_autoplace no) (hide yes) (effects (font (size 1.27 1.27)))) (property "Description" "" (at 139.7 45.72 0) (show_name no) (do_not_autoplace no) (hide yes) (effects (font (size 1.27 1.27)))) (pin "1") (pin "2") (pin "3") (pin "4") (pin "5") (instances (project "IrradianceBreakout" (path "/552486ca-d81b-4f74-b370-4ec84ac435dd" (reference "J1") (unit 1)))))
+	(wire (pts (xy 134.62 40.64) (xy 132.08 40.64)) (stroke (width 0) (type default)))
+	(label "PD_K" (at 132.08 40.64 180) (effects (font (size 1.27 1.27)) (justify right bottom)))
+	(wire (pts (xy 134.62 43.18) (xy 132.08 43.18)) (stroke (width 0) (type default)))
+	(label "PD_A" (at 132.08 43.18 180) (effects (font (size 1.27 1.27)) (justify right bottom)))
+	(wire (pts (xy 134.62 45.72) (xy 132.08 45.72)) (stroke (width 0) (type default)))
+	(label "GNDA" (at 132.08 45.72 180) (effects (font (size 1.27 1.27)) (justify right bottom)))
+	(wire (pts (xy 134.62 48.26) (xy 132.08 48.26)) (stroke (width 0) (type default)))
+	(label "GNDA" (at 132.08 48.26 180) (effects (font (size 1.27 1.27)) (justify right bottom)))
+	(no_connect (at 134.62 50.8))
+	(sheet_instances (path "/" (page "1")))
 	(embedded_fonts no)
 )

Commit message: updates
Other:
- note added: ":("
- note added: "Vishay BPW34 / BPW34 Undecided"
- note removed: "Same Nano-Fit 1x5 as the main board J. BRK_DET tied to GNDA here (main board reads low = present). Shield not connected here (terminated on the main board only)."
- note removed: "Vishay BPW34 / BPW34S, 430-1100 nm, 7.5 mm2. Top side, centred on the window. Assign the footprint once the exact package is picked."
- moved on the sheet: D1, J1

Commit message: check breakout board layout
Parts:
- removed D1: BPW34, symbol BlackBody:BPW34
- added C1: 10u, Capacitor_SMD:C_0805_2012Metric_Pad1.18x1.45mm_HandSolder, symbol Device:C
- added C2: 100n, Capacitor_SMD:C_0603_1608Metric_Pad1.08x0.95mm_HandSolder, symbol Device:C
- added D1: Red, LED_SMD:LED_0603_1608Metric, symbol Device:LED
- added D2: D5V0P4UR6SO-7, LHRS_ICs:D5V0P4UR6SO-7, symbol lhrs_ics:D5V0P4UR6SO-7
- added Q1: DMP3099L, Package_TO_SOT_SMD:SOT-23, symbol BlackBody:DMP3099L
- added R2, R3: 2.2k, Resistor_SMD:R_0603_1608Metric_Pad0.98x0.95mm_HandSolder, symbol Device:R
- added R4: 10k, Resistor_SMD:R_0603_1608Metric_Pad0.98x0.95mm_HandSolder, symbol Device:R
- added R5: 1k, Resistor_SMD:R_0603_1608Metric_Pad0.98x0.95mm_HandSolder, symbol Device:R
- added U1: TSL25911FN, OptoDevice:AMS_TSL25911FN, symbol Sensor_Optical:TSL25911FN
Connections:
- net GND: now reaches J1.5 (Pin_5)
- net GND: now also C1.2, C2.2, D1.1 (K), D2.2, U1.3 (GND)
- net GNDA renamed ALS_INT
- net ALS_INT: now also D2.6, Q1.1 (G), R4.2, U1.2 (INT); no longer J1.3 (Pin_3)
- net PD_A renamed SDA
- net SDA: now also D2.1, R2.2, U1.6 (SDA)
- net PD_K renamed +3.3V
- net +3.3V: now also C1.1, C2.1, D2.5, Q1.2 (S), R2.1, R3.1, R4.1, U1.5 (VDD)
- new net: Q1.3 (D), R5.1
- new net: D1.2 (A), R5.2
- new net SCL: D2.3, J1.3 (Pin_3), R3.2, U1.1 (SCL)
Other:
- note added: "+3.3V"
- note added: "Ambient Light Sensor"
- note added: "ESD Protection"
- note added: "GND"
- note added: "I2C Pull-ups"
- note added: "Interrupt LED"
- note added: "Lights while INT is low"
- note added: "Pmos"
- note added: "SCL"
- note added: "SDA"
- note added: "~{INT}"
- note removed: ":("
- note removed: "Photodiode"
- note removed: "Vishay BPW34 / BPW34 Undecided"

Commit message: Main board placement + silkscreen, breakout ground plane, DRC rule updates
- Grouped placement and condensed outline (2 mm rounded corners)
- Silkscreen refs moved next to their parts, pin labels added
- Interrupt removed from main board and breakout (test point instead)
- Breakout: B.Cu ground plane + stitching vias
- Default clearance / hole clearance lowered to 0.15 mm
Parts:
- removed D1: Red, LED_SMD:LED_0603_1608Metric, symbol Device:LED
- removed Q1: DMP3099L, Package_TO_SOT_SMD:SOT-23, symbol BlackBody:DMP3099L
- removed R5: 1k, Resistor_SMD:R_0603_1608Metric_Pad0.98x0.95mm_HandSolder, symbol Device:R
- added TP1: INT, TestPoint:TestPoint_Pad_D1.5mm, symbol Connector:TestPoint
Connections:
- net ALS_INT: now also TP1.1; no longer D2.6, J1.4 (Pin_4)
- net GND: now also J1.3 (Pin_3); no longer J1.5 (Pin_5)
- net SCL: now also D2.6, J1.5 (Pin_5); no longer D2.3, J1.3 (Pin_3)
- no-connect marks 1 -> 4
Other:
- note added: "INT Test Point"
- note removed: "+3.3V"
- note removed: "GND"
- note removed: "Interrupt LED"
- note removed: "Lights while INT is low"
- note removed: "Pmos"
- note removed: "SCL"
- note removed: "SDA"
- note removed: "~{INT}"
- moved on the sheet: J1
